File: KiCad/SaintSays.kicad_pcb (KiCad board)
At the start: 2 copper layers, 20 x 20 mm, 14 parts, among them SW1 SW_Push, SW2 SW_Push, SW3 SW_Push, SW4 SW_Push, U1 ATtiny84A-SS

Commit message: Adding V3 code and KiCad
Parts:
- renumbered D1 to 1, D2 to 2, D3 to 4, D4 to 8
Changed lines of the file:
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@@
 		(descr "LED SMD 1206 (3216 Metric), square (rectangular) end terminal, IPC_7351 nominal, (Body size source: http://www.tortai-tech.com/upload/download/2011102023233369053.pdf), generated with kicad-footprint-generator")
 		(tags "LED handsolder")
-		(property "Reference" "D4"
+		(property "Reference" "8"
 			(at -1.7125 1.75 180)
 			(layer "F.SilkS")
@@
 		(descr "LED SMD 1206 (3216 Metric), square (rectangular) end terminal, IPC_7351 nominal, (Body size source: http://www.tortai-tech.com/upload/download/2011102023233369053.pdf), generated with kicad-footprint-generator")
 		(tags "LED handsolder")
-		(property "Reference" "D1"
+		(property "Reference" "1"
 			(at -1.5875 1.75 180)
 			(layer "F.SilkS")
@@
 		(descr "LED SMD 1206 (3216 Metric), square (rectangular) end terminal, IPC_7351 nominal, (Body size source: http://www.tortai-tech.com/upload/download/2011102023233369053.pdf), generated with kicad-footprint-generator")
 		(tags "LED handsolder")
-		(property "Reference" "D2"
+		(property "Reference" "2"
 			(at 1.71 -1.7 0)
 			(layer "F.SilkS")
@@
 		(descr "LED SMD 1206 (3216 Metric), square (rectangular) end terminal, IPC_7351 nominal, (Body size source: http://www.tortai-tech.com/upload/download/2011102023233369053.pdf), generated with kicad-footprint-generator")
 		(tags "LED handsolder")
-		(property "Reference" "D3"
+		(property "Reference" "4"
 			(at 1.81 -1.65 0)
 			(layer "F.SilkS")
